File: HW/databank.brd (EAGLE design)
At the start: 64.5 x 45.7 mm, 33 parts

Commit message: Finished design
Parts:
- removed LED1, LED2: (no value), led:CHIP-LED0603
- removed R11, R22: (no value), rcl:R0603
- added R18, R21, R23, R24, R25: 33, rcl:R0603
- R1, R12, R13, R14, R15, R16, R17, R2, R3, R4, R5, R6: value 100K -> 10K
- moved C9 206.0 mm to (40.6, 41.3), flipped to the bottom, turned to 270 degrees
- moved R14 200.4 mm to (67.3, 38.7), flipped to the bottom
- moved C6 199.8 mm to (67.3, 36.2), flipped to the bottom, turned to 180 degrees
- moved R15 197.3 mm to (64.1, 41.9), flipped to the bottom, turned to 270 degrees
- moved C5 197.1 mm to (38.1, 41.3), flipped to the bottom, turned to 270 degrees
- moved C7 192.8 mm to (35.6, 41.3), flipped to the bottom, turned to 270 degrees
- moved R19 192.0 mm to (61.0, 38.1), flipped to the bottom, turned to 270 degrees
- moved R16 192.0 mm to (61.0, 41.9), flipped to the bottom, turned to 270 degrees
- moved R20 191.0 mm to (64.1, 38.1), flipped to the bottom, turned to 270 degrees
- moved R12 189.2 mm to (38.1, 36.8), flipped to the bottom, turned to 90 degrees
- moved C8 185.7 mm to (34.9, 36.8), flipped to the bottom, turned to 270 degrees
- moved R13 179.7 mm to (33.0, 33.0), flipped to the bottom, turned to 270 degrees
- moved R17 174.9 mm to (41.9, 36.8), flipped to the bottom
- moved C4 169.7 mm to (50.2, 42.5), turned to 180 degrees
- moved C3 153.4 mm to (50.2, 38.7), turned to 180 degrees
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Connections:
- removed net N$1: LED1.C, R11.2
- removed net N$10: LED2.C, R22.2
- removed net SD0_STAT: R11.1, U$1.GPIO@1
- removed net SD1_STAT: R22.1, U$1.GPIO@2
- new net N$11: R23.2, U$1.TIM@8
- new net N$12: R24.2, U$1.TIM@7
- new net N$13: R25.2, U$1.TIM@6
- new net N$8: R21.2, U$1.TIM@10
- new net N$9: R18.2, U$1.TIM@9
- net +3V3: no longer LED1.A, LED2.A
- net FLASH_!HOLD: now also R21.1; no longer U$1.TIM@9
- net SD0_!CD: now also R23.1, R8.1; no longer C4.1, U$1.TIM@7
- net SD0_!WP: now also C4.1, R25.1; no longer R8.1, U$1.TIM@5
- net SD1_!CD: now also R18.1, R19.1; no longer C8.1, U$1.TIM@8
- net SD1_!WP: now also C8.1, R24.1; no longer R19.1, U$1.TIM@6
Routing:
- net GND: track 0.00 -> 125.4 mm, vias 0 -> 12
- net +3V3: track 0.00 -> 107.9 mm, vias 0 -> 10
- net SCLK: track 0.00 -> 87.5 mm, vias 0 -> 7
- net SD1_!CD: track 0.00 -> 72.6 mm, vias 0 -> 3
- net SD0_!WP: track 0.00 -> 72.2 mm, vias 0 -> 2
- net MISO: track 0.00 -> 69.9 mm, vias 0 -> 6
- net MOSI: track 0.00 -> 67.3 mm, vias 0 -> 5
- net SD0_!CD: track 0.00 -> 56.9 mm, vias 0 -> 1
- net SD1_!WP: track 0.00 -> 55.6 mm, vias 0 -> 6
- net FLASH_!CS: track 0.00 -> 52.0 mm, vias 0 -> 4
- net SD1_!CS: track 0.00 -> 46.7 mm, vias 0 -> 2
- net FLASH_!HOLD: track 0.00 -> 41.0 mm, vias 0 -> 5
- net N$6: track 0.00 -> 39.5 mm, vias 0 -> 3
- net SD0_!CS: track 0.00 -> 31.3 mm, vias 0 -> 4
- net N$2: track 0.00 -> 11.5 mm, vias 0 -> 2
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Other:
- board size 64.5 x 45.7 mm -> 50.8 x 38.1 mm
- board text added: "Data Bank"
- board text removed: "Interacto"
