File: HW/databank.sch (EAGLE design)
At the start: 33 parts

Commit message: Finished design
Parts:
- removed LED1, LED2: (no value), led:LEDCHIP-LED0603
- removed R11, R22: (no value), rcl:R-US_R0603
- added R18, R21, R23, R24, R25: 33, rcl:R-US_R0603
- C1, C3, C4, C5, C7, C8, C9: MPN (none) -> VJ0603V104ZXXCW1BC
- C2, C6: MPN (none) -> LMK107BBJ106MALT
- R1, R12, R13, R14, R15, R16, R17, R2, R3, R4, R5, R6: value 100K -> 10K; MPN (none) -> WR06X1002FTL
- R19, R20, R8, R9: MPN (none) -> WR06X1002FTL
- U$2, U$3: MPN (none) -> 101-00405-75
- U$4: MPN (none) -> MX25L25635E
Connections:
- removed net N$1: LED1.C, R11.2
- removed net N$10: LED2.C, R22.2
- removed net SD0_STAT: R11.1, U$1.GPIO@1
- removed net SD1_STAT: R22.1, U$1.GPIO@2
- new net N$11: R23.2, U$1.TIM@8
- new net N$12: R24.2, U$1.TIM@7
- new net N$13: R25.2, U$1.TIM@6
- new net N$8: R21.2, U$1.TIM@10
- new net N$9: R18.2, U$1.TIM@9
- net +3V3: no longer LED1.A, LED2.A
- net FLASH_!HOLD: now also R21.1; no longer U$1.TIM@9
- net SD0_!CD: now also R23.1, R8.1; no longer C4.1, U$1.TIM@7
- net SD0_!WP: now also C4.1, R25.1; no longer R8.1, U$1.TIM@5
- net SD1_!CD: now also R18.1, R19.1; no longer C8.1, U$1.TIM@8
- net SD1_!WP: now also C8.1, R24.1; no longer R19.1, U$1.TIM@6
Other:
- moved on the sheet: C9, U$1, U$4
